File: pcb/yak40_main/yak40_main.kicad_pcb (KiCad board)
At the start: 2 copper layers, 285 x 94.5 mm, 136 parts, among them J1 Conn_01x04, J2 Conn_01x03_Pin, SW1 SW_Push, SW10 SW_Push, SW11 SW_Push, SW12 SW_Push, SW13 SW_Push, SW14 SW_Push, SW15 SW_Push, SW16 SW_Push, SW17 SW_Push, SW18 SW_Push, SW19 SW_Push, SW2 SW_Push, SW20 SW_Push, SW21 SW_Push, SW22 SW_Push, SW23 SW_Push, SW24 SW_Push, SW25 SW_Push, SW26 SW_Push, SW27 SW_Push, SW28 SW_Push, SW29 SW_Push, SW3 SW_Push, SW30 SW_Push, SW31 SW_Push, SW32 SW_Push, SW33 SW_Push, SW34 SW_Push, SW35 SW_Push, SW36 SW_Push, SW37 SW_Push, SW38 SW_Push, SW39 SW_Push, SW4 SW_Push, SW40 SW_Push, SW41 SW_Push, SW42 SW_Push, SW43 SW_Push, SW44 SW_Push, SW45 SW_Push, SW46 SW_Push, SW47 SW_Push, SW48 SW_Push, SW49 SW_Push, SW5 SW_Push, SW50 SW_Push, SW51 SW_Push, SW52 SW_Push, SW53 SW_Push, SW54 SW_Push, SW55 SW_Push, SW6 SW_Push, SW7 SW_Push, SW8 SW_Push, SW9 SW_Push, U1 NCP1117-3.3_SOT223, U2 RP2040, U3 W25Q128JVS, Y1 Crystal

Commit message: Update pcb
Parts:
- added C17: 22p, Capacitor_SMD:C_0402_1005Metric, B.Cu at (138.2, 62.4)
- added C18: 22p, Capacitor_SMD:C_0402_1005Metric, B.Cu at (135.3, 59.6)
- C10, C9: value 10u -> 1u
- D1, D10, D11, D12, D13, D15, D16, D17, D18, D19, D2, D20, D21, D22, D23, D24, D25, D26, D27, D28, D29, D3, D30, D31, D32, D33, D34, D35, D36, D37, D38, D39, D4, D42, D43, D44, D45, D46, D47, D48, D49, D5, D6, D7, D8, D9: footprint Diode_SMD:D_1206_3216Metric_Pad1.42x1.75mm_HandSolder -> Diode_SMD:D_SOD-123
- SW54, SW55: footprint Button_Switch_SMD:SW_Push_1P1T_NO_Vertical_Wuerth_434133025816 -> Button_Switch_SMD:SW_Push_1P1T_XKB_TS-1187A
- U1: value NCP1117-3.3_SOT223 -> XC6206PxxxMR; footprint Package_TO_SOT_SMD:SOT-223-3_TabPin2 -> Package_TO_SOT_SMD:SOT-23-3
- U3: footprint Package_SON:WSON-8-1EP_6x5mm_P1.27mm_EP3.4x4.3mm -> Package_SO:SOIC-8_5.23x5.23mm_P1.27mm
- Y1: value Crystal -> 12MHz; footprint Crystal:Resonator_SMD_Murata_CSTxExxV-3Pin_3.0x1.1mm_HandSoldering -> Crystal:Crystal_SMD_3225-4Pin_3.2x2.5mm
- moved H7 27.9 mm to (248.6, 25.0)
- moved D48 22.7 mm to (197.4, 77.9)
- moved D38 20.4 mm to (240.0, 54.6)
- moved H1 17.7 mm to (26.3, 24.0)
- moved R5 7.59 mm to (147.2, 45.2), turned to 90 degrees
- moved R4 6.39 mm to (148.4, 45.2), turned to -90 degrees
- moved C16 5.24 mm to (148.4, 37.4), turned to 90 degrees
- moved C9 4.73 mm to (128.0, 37.4), turned to -90 degrees
- moved C15 4.29 mm to (147.2, 37.4), turned to 90 degrees
- moved C10 3.56 mm to (133.1, 37.4), turned to 90 degrees
- moved SW55 2.98 mm to (132.8, 71.6), turned to 90 degrees
- moved SW11 2.53 mm to (227.3, 14.1)
- moved J2 2.39 mm to (138.8, 66.1)
- moved D39 2.38 mm to (260.9, 54.6)
- moved SW12 2.09 mm to (246.3, 14.5)
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Connections:
- R6 pad 1: XOUT -> /XTAL_O
- R6 pad 2: Net-(R6-Pad2) -> XOUT
- Y1 pad 1: XIN -> /XTAL_O
- Y1 pad 3: Net-(R6-Pad2) -> XIN
Routing:
- net Net-(D48-A): track 11.0 -> 34.2 mm
- net Net-(D39-A): track 10.5 -> 33.6 mm
- net Net-(D38-A): track 11.0 -> 33.3 mm
- net Column13: track 215.3 -> 203.8 mm
- net QSPI_SD3: track 6.69 -> 17.4 mm
- net QSPI_SCLK: track 5.62 -> 15.5 mm
- net QSPI_SD0: track 4.66 -> 12.5 mm
- net QSPI_SS: track 18.8 -> 11.7 mm
- net QSPI_SD1: track 14.4 -> 7.53 mm
- net QSPI_SD2: track 13.2 -> 6.70 mm
- net ~{BOOT}: track 38.1 -> 33.0 mm
- net XIN: track 6.38 -> 9.86 mm
- net Row2: track 268.8 -> 272.3 mm
- net /XTAL_O: track 0.00 -> 3.15 mm
- net Net-(R6-Pad2): track 2.42 -> 0.00 mm
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Other:
- board size 285 x 94.5 mm -> 285 x 93.5 mm
- board text added: "v.20231201"

Commit message: Update PCB to be cheaper
Routing:
- net GND: track 2.84 -> 34.4 mm, vias 128 -> 134
Other:
- outline, holes or cut-outs redrawn
- board text added: "Designed by kuriki-sasa"
- board text added: "JLCJLCJLCJLC"
- board text removed: "Designed by kurikisasa"
- board text removed: "Yak40"
- board text removed: "v.20231201"

Commit message: Support LED and rotary encoders
Parts:
- added J3: Conn_01x03_Pin, Connector_PinHeader_2.54mm:PinHeader_1x03_P2.54mm_Vertical, B.Cu at (-8.88, 40.6)
- added Q1: BSS138, Package_TO_SOT_SMD:SOT-23, B.Cu at (115.3, 60.9)
- added R7: 1k, Resistor_SMD:R_0402_1005Metric, B.Cu at (115.7, 63.4)
- added R8: 560, Resistor_SMD:R_0603_1608Metric, B.Cu at (111.1, 57.9)
- SW45, SW46: value SW_Push -> RotaryEncoder_Switch; footprint MX_Hotswap:MX-Hotswap-1U -> kicad-libs:SW_Cherry_MX_1.00u_Kailh_EC12
- moved D46 40.4 mm to (126.5, 107.8)
- moved SW32 25.4 mm to (104.9, 84.6)
- moved C4 25.4 mm to (115.6, 68.4)
- moved SW47 25.4 mm to (163.7, 99.2)
- moved R4 25.4 mm to (133.0, 65.4)
- moved SW9 25.4 mm to (172.6, 39.6)
- moved D27 25.4 mm to (10.2, 74.7)
- moved SW51 25.4 mm to (89.8, 101.3)
- moved D32 25.4 mm to (112.7, 88.0)
- moved SW24 25.4 mm to (199.3, 54.3)
- moved SW42 25.4 mm to (20.1, 91.8)
- moved SW46 25.4 mm to (135.6, 104.2)
- moved SW39 25.4 mm to (256.7, 72.7)
- moved C2 25.4 mm to (121.5, 64.1)
- moved SW10 25.4 mm to (191.3, 36.3)
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Connections:
- U2 pad 13: unconnected-(U2-GPIO10-Pad13) -> Rotary2A
- U2 pad 14: unconnected-(U2-GPIO11-Pad14) -> Rotary2B
- U2 pad 15: unconnected-(U2-GPIO12-Pad15) -> Rotary1A
- U2 pad 16: unconnected-(U2-GPIO13-Pad16) -> Rotary1B
- U2 pad 38: unconnected-(U2-GPIO26_ADC0-Pad38) -> LED3V3
Routing:
- net LED5V: track 0.00 -> 128.8 mm
- net +5V: track 9.70 -> 134.3 mm
- net Rotary1B: track 0.00 -> 38.8 mm
- net Rotary1A: track 0.00 -> 34.2 mm
- net Rotary2A: track 0.00 -> 31.8 mm
- net Rotary2B: track 0.00 -> 26.6 mm
- net Column7: track 81.7 -> 98.8 mm
- net Column6: track 90.3 -> 103.4 mm
- net Net-(D45-A): track 6.45 -> 17.8 mm, vias 0 -> 1
- net LED3V3: track 0.00 -> 11.1 mm
- net +3V3: track 98.3 -> 106.1 mm
- net Net-(D46-A): track 6.45 -> 13.3 mm, vias 0 -> 1
- net Row4: track 255.3 -> 260.7 mm
- net Column1: track 164.5 -> 169.3 mm
- net Row1: track 280.9 -> 277.7 mm, vias 0 -> 2
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Other:
- board text removed: "JLCJLCJLCJLC"
